File: secondPCB/FreeWatch/FreeWatch.kicad_sch (KiCad schematic)
At the start: 5 parts, among them U1 MAX30102, U2 DS3231MZ, U3 MCP23008-xSO

Commit message: moving on
Parts:
- added U4: APDS-9960, APDS-9960:APDS-9960, symbol APDS-9960:APDS-9960
- R1, R2: footprint (none) -> Resistor_SMD:R_0603_1608Metric
Connections:
- net +3V3: now also U4.5 (LEDA), U4.8 (VDD)
- net GND: now also U4.6 (GND)
- net SCL: now also U4.7 (SCL)
- net SDA: now also U4.1 (SDA)
- new net: U4.3 (LDR), U4.4 (LEDK)
Changed lines of the file:
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@@
   (junction (at 200.66 119.38) (diameter 0) (color 0 0 0 0)
   )
+  (junction (at 60.96 153.67) (diameter 0) (color 0 0 0 0)
+  )
   (junction (at 218.44 128.27) (diameter 0) (color 0 0 0 0)
   )
@@
     (stroke (width 0) (type default))
   )
+  (wire (pts (xy 60.96 163.83) (xy 74.93 163.83))
+    (stroke (width 0) (type default))
+  )
   (wire (pts (xy 193.04 101.6) (xy 205.74 101.6))
     (stroke (width 0) (type default))
@@
     (stroke (width 0) (type default))
   )
+  (wire (pts (xy 60.96 153.67) (xy 60.96 163.83))
+    (stroke (width 0) (type default))
+  )
+  (wire (pts (xy 100.33 156.21) (xy 105.41 156.21))
+    (stroke (width 0) (type default))
+  )
   (wire (pts (xy 66.04 107.95) (xy 76.2 107.95))
     (stroke (width 0) (type default))
@@
     (stroke (width 0) (type default))
   )
-  (wire (pts (xy 154.94 87.63) (xy 154.94 96.52))
+  (wire (pts (xy 154.94 85.09) (xy 154.94 96.52))
     (stroke (width 0) (type default))
   )
@@
     (stroke (width 0) (type default))
   )
+  (wire (pts (xy 100.33 163.83) (xy 114.3 163.83))
+    (stroke (width 0) (type default))
+  )
+  (wire (pts (xy 105.41 156.21) (xy 105.41 153.67))
+    (stroke (width 0) (type default))
+  )
   (wire (pts (xy 218.44 128.27) (xy 218.44 130.81))
     (stroke (width 0) (type default))
@@
     (stroke (width 0) (type default))
   )
+  (wire (pts (xy 71.12 158.75) (xy 74.93 158.75))
+    (stroke (width 0) (type default))
+  )
+  (wire (pts (xy 100.33 161.29) (xy 114.3 161.29))
+    (stroke (width 0) (type default))
+  )
   (wire (pts (xy 200.66 114.3) (xy 200.66 116.84))
     (stroke (width 0) (type default))
@@
     (stroke (width 0) (type default))
   )
+  (wire (pts (xy 100.33 153.67) (xy 105.41 153.67))
+    (stroke (width 0) (type default))
+  )
   (wire (pts (xy 58.42 45.72) (xy 58.42 50.8))
     (stroke (width 0) (type default))
@@
     (stroke (width 0) (type default))
   )
+  (wire (pts (xy 60.96 152.4) (xy 60.96 153.67))
+    (stroke (width 0) (type default))
+  )
   (wire (pts (xy 218.44 124.46) (xy 218.44 128.27))
+    (stroke (width 0) (type default))
+  )
+  (wire (pts (xy 60.96 153.67) (xy 74.93 153.67))
     (stroke (width 0) (type default))
   )
@@
     )
   )
-  (global_label "VSYS" (shape input) (at 152.4 90.17 180) (fields_autoplaced)
-    (effects (font (size 1.27 1.27)) (justify right))
-    (property "Intersheetrefs" "${INTERSHEET_REFS}" (at 144.898 90.17 0)
-      (effects (font (size 1.27 1.27)) (justify right) hide)
+  (global_label "VSYS" (shape input) (at 152.4 90.17 90) (fields_autoplaced)
+    (effects (font (size 1.27 1.27)) (justify left))
+    (property "Intersheetrefs" "${INTERSHEET_REFS}" (at 152.4 82.668 90)
+      (effects (font (size 1.27 1.27)) (justify left) hide)
     )
   )
@@
     )
   )
+  (global_label "SCL" (shape input) (at 114.3 161.29 0) (fields_autoplaced)
+    (effects (font (size 1.27 1.27)) (justify left))
+    (property "Intersheetrefs" "${INTERSHEET_REFS}" (at 120.7134 161.29 0)
+      (effects (font (size 1.27 1.27)) (justify left) hide)
+    )
+  )
   (global_label "SCL" (shape input) (at 58.42 50.8 0) (fields_autoplaced)
     (effects (font (size 1.27 1.27)) (justify left))
@@
     )
   )
+  (global_label "SDA" (shape input) (at 114.3 163.83 0) (fields_autoplaced)
+    (effects (font (size 1.27 1.27)) (justify left))
+    (property "Intersheetrefs" "${INTERSHEET_REFS}" (at 120.7739 163.83 0)
+      (effects (font (size 1.27 1.27)) (justify left) hide)
+    )
+  )
   (global_label "SCL" (shape input) (at 132.08 101.6 180) (fields_autoplaced)
     (effects (font (size 1.27 1.27)) (justify right))
@@
     )
   )
-  (symbol (lib_id "power:+3V3") (at 154.94 87.63 0) (unit 1)
-    (in_bom yes) (on_board yes) (dnp no) (fields_autoplaced)
-    (property "Reference" "#PWR07" (at 154.94 91.44 0)
-      (effects (font (size 1.27 1.27)) hide)
-    )
-    (property "Value" "+3V3" (at 154.94 82.55 0)
-      (effects (font (size 1.27 1.27)))
-    )
-    (property "Footprint" "" (at 154.94 87.63 0)
-      (effects (font (size 1.27 1.27)) hide)
-    )
-    (property "Datasheet" "" (at 154.94 87.63 0)
+  (symbol (lib_id "power:+3V3") (at 154.94 85.09 0) (unit 1)
+    (in_bom yes) (on_board yes) (dnp no) (fields_autoplaced)
+    (property "Reference" "#PWR07" (at 154.94 88.9 0)
+      (effects (font (size 1.27 1.27)) hide)
+    )
+    (property "Value" "+3V3" (at 154.94 80.01 0)
+      (effects (font (size 1.27 1.27)))
+    )
+    (property "Footprint" "" (at 154.94 85.09 0)
+      (effects (font (size 1.27 1.27)) hide)
+    )
+    (property "Datasheet" "" (at 154.94 85.09 0)
       (effects (font (size 1.27 1.27)) hide)
     )
@@
     )
   )
+  (symbol (lib_id "power:+3V3") (at 60.96 152.4 0) (unit 1)
+    (in_bom yes) (on_board yes) (dnp no) (fields_autoplaced)
+    (property "Reference" "#PWR010" (at 60.96 156.21 0)
+      (effects (font (size 1.27 1.27)) hide)
+    )
+    (property "Value" "+3V3" (at 60.96 147.32 0)
+      (effects (font (size 1.27 1.27)))
+    )
+    (property "Footprint" "" (at 60.96 152.4 0)
+      (effects (font (size 1.27 1.27)) hide)
+    )
+    (property "Datasheet" "" (at 60.96 152.4 0)
+      (effects (font (size 1.27 1.27)) hide)
+    )
+    (pin "1")
+    (instances
+      (project "FreeWatch"
+        (path "/fd27948c-d175-4cf4-b2a1-fcdef57001f9"
+          (reference "#PWR010") (unit 1)
+        )
+      )
+    )
+  )
   (symbol (lib_id "power:+3V3") (at 218.44 88.9 0) (unit 1)
     (in_bom yes) (on_board yes) (dnp no) (fields_autoplaced)
@@
       (effects (font (size 1.27 1.27)) (justify left))
     )
-    (property "Footprint" "" (at 56.642 41.91 90)
+    (property "Footprint" "Resistor_SMD:R_0603_1608Metric" (at 56.642 41.91 90)
       (effects (font (size 1.27 1.27)) hide)
     )
@@
       (effects (font (size 1.27 1.27)) (justify left))
     )
-    (property "Footprint" "" (at 70.612 41.91 90)
+    (property "Footprint" "Resistor_SMD:R_0603_1608Metric" (at 70.612 41.91 90)
       (effects (font (size 1.27 1.27)) hide)
     )
@@
         (path "/fd27948c-d175-4cf4-b2a1-fcdef57001f9"
           (reference "#PWR05") (unit 1)
+        )
+      )
+    )
+  )
+  (symbol (lib_id "power:GND") (at 71.12 158.75 270) (unit 1)
+    (in_bom yes) (on_board yes) (dnp no) (fields_autoplaced)
+    (property "Reference" "#PWR011" (at 64.77 158.75 0)
+      (effects (font (size 1.27 1.27)) hide)
+    )
+    (property "Value" "GND" (at 67.31 158.75 90)
+      (effects (font (size 1.27 1.27)) (justify right))
+    )
+    (property "Footprint" "" (at 71.12 158.75 0)
+      (effects (font (size 1.27 1.27)) hide)
+    )
+    (property "Datasheet" "" (at 71.12 158.75 0)
+      (effects (font (size 1.27 1.27)) hide)
+    )
+    (pin "1")
+    (instances
+      (project "FreeWatch"
+        (path "/fd27948c-d175-4cf4-b2a1-fcdef57001f9"
+          (reference "#PWR011") (unit 1)
         )
       )
@@
         )
       )
+    )
+  )
+  (symbol (lib_id "APDS-9960:APDS-9960") (at 87.63 158.75 0) (unit 1)
+    (in_bom yes) (on_board yes) (dnp no) (fields_autoplaced)
+    (property "Reference" "U4" (at 87.63 146.05 0)
+      (effects (font (size 1.27 1.27)))
+    )
+    (property "Value" "APDS-9960" (at 87.63 148.59 0)
+      (effects (font (size 1.27 1.27)))
+    )
+    (property "Footprint" "APDS-9960:APDS-9960" (at 87.63 158.75 0)
+      (effects (font (size 1.27 1.27)) (justify bottom) hide)
+    )
+    (property "Datasheet" "" (at 87.63 158.75 0)
+      (effects (font (size 1.27 1.27)) hide)
+    )
+    (property "PROD_ID" "SEN-12005" (at 87.63 158.75 0)
+      (effects (font (size 1.27 1.27)) (justify bottom) hide)
+    )
+    (pin "1")
+    (pin "2")
+    (pin "3")
+    (pin "4")
+    (pin "5")
+    (pin "6")
+    (pin "7")
+    (pin "8")
+    (instances
+      (project "FreeWatch"
+        (path "/fd27948c-d175-4cf4-b2a1-fcdef57001f9"
+          (reference "U4") (unit 1)
+        )
+      )
